File: CJ125 Circuit Design/CJ125 Circuit Design.kicad_sch (KiCad schematic)
At the start: 15 parts, among them U1 CJ125

Commit message: updated a bunch of cj125 stuff
Parts:
- added C7: 33n, symbol Device:C
- added C8: 2.2n, symbol Device:C
- added C9: 10n, symbol Device:C
- added J1: 2x3 Connector to ECU, symbol Connector_Generic:Conn_02x03_Odd_Even
- added J2: STLink, symbol Connector_Generic:Conn_02x10_Odd_Even
- added J3: 2x3 Connector to O2 Sensor, symbol Connector_Generic:Conn_02x03_Odd_Even
- added Q1: NMOS, symbol Simulation_SPICE:NMOS
- added R10: 100K, symbol Device:R
- added R9: 301, symbol Device:R
- added U2: LM1117DT-5.0, Package_TO_SOT_SMD:TO-252-3_TabPin2, symbol Regulator_Linear:LM1117DT-5.0
- added U3: STM32F103CBTx, Package_QFP:LQFP-48_7x7mm_P0.5mm, symbol MCU_ST_STM32F1:STM32F103CBTx
- added U4: CAN Tranceiver, Package_SO:SOP-8_6.62x9.15mm_P2.54mm, symbol Interface_CAN_LIN:ISO1050DUB
- R1: value R -> 31.6K
Connections:
- net GND: now also C7.1, C8.1, C9.2, J1.6 (Pin_6), J2.10 (Pin_10), J2.12 (Pin_12), J2.14 (Pin_14), J2.15 (Pin_15), J2.16 (Pin_16), J2.18 (Pin_18), J2.20 (Pin_20), J2.4 (Pin_4), J2.6 (Pin_6), J2.8 (Pin_8), U2.1 (GND), U3.23 (VSS), U3.35 (VSS), U3.47 (VSS), U3.8 (VSSA), U4.4 (GND1), U4.5 (GND2)
- net UN: now reaches R7.2
- net UN: now also C8.2, J3.1 (Pin_1), R10.1
- net +12V: now reaches C6.1, U1.1 (UB)
- net +12V: now also J1.1 (Pin_1), J3.5 (Pin_5), U2.3 (VI)
- net at C5.1, U1.17 (VCC): now also U2.2 (VO)
- net UA_ADC: now reaches C4.1, U1.21 (UA)
- net UA_ADC: now also U3.19 (PB1)
- net at R8.1: now also Q1.1 (D)
- net IA: now reaches R5.1, R6.1, U1.4 (IA)
- net IA: now also J3.3 (Pin_3)
- net IP: now reaches R6.2, U1.3 (IP)
- net IP: now also J3.6 (Pin_6)
- net UR_ADC: now reaches C3.1, U1.12 (UR)
- net UR_ADC: now also U3.18 (PB0)
- net SPI_SCK: now reaches U1.13 (SCK)
- net SPI_SCK: now also U3.15 (PA5)
- net SPI_MISO: now reaches U1.14 (MISO)
- net SPI_MISO: now also U3.16 (PA6)
- net SPI_MOSI: now reaches U1.15 (MOSI)
- net SPI_MOSI: now also U3.17 (PA7)
- net SPI_NSS: now reaches U1.16 (~{SS})
- net SPI_NSS: now also U3.14 (PA4)
- net VM: now reaches U1.18 (VM)
- net VM: now also J3.4 (Pin_4), R9.1
- net at U1.2 (UN): now also C7.2, R10.2
- net HTR_CTRL: now reaches U1.6 (DIAHG)
- net HTR_CTRL: now also Q1.2 (G), U3.31 (PA10)
- net at U1.9 (RS): now also R9.2
- new net +3V3: C9.1, J2.1 (Pin_1), J2.2 (Pin_2), U3.1 (VBAT), U3.24 (VDD), U3.36 (VDD), U3.48 (VDD), U3.9 (VDDA), U4.1 (VCC1)
- new net +5V: U4.8 (VCC2)
- new net CANH: J1.2 (Pin_2), U4.7 (CANH)
- new net CANL: J1.4 (Pin_4), U4.6 (CANL)
- new net CAN_RX: U3.32 (PA11), U4.2 (RXD)
- new net CAN_TX: U3.33 (PA12), U4.3 (TXD)
- new net Heater-: J3.2 (Pin_2), Q1.3 (S)
- new net SWCLK: J2.9 (Pin_9), U3.37 (PA14)
- new net SWDIO: J2.7 (Pin_7), U3.34 (PA13)
- new net SWO: J2.13 (Pin_13), U3.39 (PB3)
- no-connect marks 0 -> 6
Other:
- moved on the sheet: C1, C2, C3, C4, C5, C6, R1, R2, R3, R4, R5, R6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

Commit message: added a bunch of stuff for hte board
Parts:
- removed Q1: NMOS, symbol Simulation_SPICE:NMOS
- removed U4: CAN Tranceiver, Package_SO:SOP-8_6.62x9.15mm_P2.54mm, symbol Interface_CAN_LIN:ISO1050DUB
- added C10, C11: 10u, Capacitor_SMD:C_0603_1608Metric, symbol Device:C
- added C12, C13, C14, C15, C16: 10n, Capacitor_SMD:C_0603_1608Metric, symbol Device:C
- added C17: 100nF, Capacitor_SMD:C_0603_1608Metric, symbol Device:C
- added C18: 1n, Capacitor_SMD:C_0603_1608Metric, symbol Device:C
- added D1: D_TVS_Dual_AAC, Package_TO_SOT_SMD:SOT-23, symbol Device:D_TVS_Dual_AAC
- added FL1: Filter_1812CAN, Inductor_SMD:L_CommonModeChoke_Coilcraft_1812CAN, symbol Motor_Driver_Components:Filter_1812CAN
- added IC1: SI2302CDS-T1-BE3, SOT95P237X112-3N, symbol SI2302CDS-T1-BE3:SI2302CDS-T1-BE3
- added R11: 120, Resistor_SMD:R_0603_1608Metric, symbol Device:R
- added U5: ISO1050DUB, Package_SO:SOP-8_6.62x9.15mm_P2.54mm, symbol Interface_CAN_LIN:ISO1050DUB
- C1, C2, C3, C4, C5, C6, C7, C8, C9: footprint (none) -> Capacitor_SMD:C_0603_1608Metric
- J1, J3: footprint (none) -> Connector_PinHeader_1.00mm:PinHeader_2x03_P1.00mm_Vertical
- J2: footprint (none) -> Connector_PinHeader_1.00mm:PinHeader_2x10_P1.00mm_Vertical
- R1, R10, R2, R3, R4, R5, R6, R7, R8, R9: footprint (none) -> Resistor_SMD:R_0603_1608Metric
- U1: footprint CJ125:SO24W -> CJ125 Circuit Data:SO24W
Connections:
- net +12V: now also J1.5 (Pin_5), C11.1; no longer J1.1 (Pin_1)
- net +3V3: now also J1.1 (Pin_1), C12.1, C13.1, C14.1, C15.1, C16.1, U5.8 (VCC2)
- net +5V: now also C5.1, U1.17 (VCC), U2.2 (VO), C10.1, C17.1, U5.1 (VCC1)
- net CANH: now also J1.4 (Pin_4), D1.2 (A2), FL1.1, R11.1; no longer J1.2 (Pin_2)
- net CANL: now also J1.2 (Pin_2), D1.1 (A1), FL1.4, R11.2; no longer J1.4 (Pin_4)
- net CAN_RX: now also U3.45 (PB8), U5.2 (RXD); no longer U3.32 (PA11)
- net CAN_TX: now also U3.46 (PB9), U5.3 (TXD); no longer U3.33 (PA12)
- net GND: now also C10.2, C11.2, C12.2, C13.2, C14.2, C15.2, C16.2, C17.2, C18.2, D1.3 (common), U5.4 (GND1), U5.5 (GND2)
- net HTR_CTRL: now also IC1.1 (G)
- net Heater-: now also IC1.2 (S)
- net UA_ADC: now also U3.12 (PA2); no longer U3.19 (PB1)
- net at R8.1: now also IC1.3 (D)
- net at U1.8 (~{RST}): now also C18.1
- new net: FL1.3, U5.6 (CANL)
- new net: FL1.2, U5.7 (CANH)
Other:
- moved on the sheet: C9, J2, R1, U2

Commit message: worked on some software but mainly just o2 board design
Parts:
- removed J1: 2x3 Connector to ECU, Connector_PinHeader_1.00mm:PinHeader_2x03_P1.00mm_Vertical, symbol Connector_Generic:Conn_02x03_Odd_Even
- removed J3: 2x3 Connector to O2 Sensor, Connector_PinHeader_1.00mm:PinHeader_2x03_P1.00mm_Vertical, symbol Connector_Generic:Conn_02x03_Odd_Even
- added J4: 1x6 O2 Connector, Connector_PinHeader_1.00mm:PinHeader_1x06_P1.00mm_Vertical, symbol Connector:Conn_01x06_Pin
- added J5: 1x6 ECU Connector, Connector_PinHeader_1.00mm:PinHeader_1x06_P1.00mm_Vertical, symbol Connector:Conn_01x06_Pin
Connections:
- net +12V: now also J4.6 (Pin_6), J5.1 (Pin_1)
- net +3V3: now also J5.6 (Pin_6)
- net CANH: now also J5.2 (Pin_2)
- net CANL: now also J5.3 (Pin_3)
- net GND: now also J5.5 (Pin_5)
- net HTR_CTRL: now also U3.21 (PB10); no longer U3.31 (PA10)
- net Heater-: now also J4.4 (Pin_4)
- net IA: now also J4.3 (Pin_3)
- net IP: now also J4.2 (Pin_2)
- net UN: now also J4.1 (Pin_1)
- net UR_ADC: now also U3.22 (PB11); no longer U3.18 (PB0)
- net VM: now also J4.5 (Pin_5)

Commit message: new board design
Parts:
- removed J4: 1x6 O2 Connector, Connector_PinHeader_1.00mm:PinHeader_1x06_P1.00mm_Vertical, symbol Connector:Conn_01x06_Pin
- added J1: 2x3 O2 Connector, CJ125 Circuit Data:MOLEX_1053101106, symbol MolexReceptacle 2x3:1053101106
- J2: footprint Connector_PinHeader_1.00mm:PinHeader_2x10_P1.00mm_Vertical -> Connector_IDC:IDC-Header_2x10_P2.54mm_Vertical
Connections:
- net +12V: now also J1.3
- net Heater-: now also J1.1
- net IA: now also J1.6
- net IP: now also J1.5
- net UN: now also J1.4
- net VM: now also J1.2
Changed lines of the file:
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@@
     (effects (font (size 1.27 1.27)) (justify left bottom))
   )
-  (label "IA" (at 33.02 91.44 0) (fields_autoplaced)
+  (label "IA" (at 45.72 116.84 0) (fields_autoplaced)
     (effects (font (size 1.27 1.27)) (justify left bottom))
   )
@@
     (effects (font (size 1.27 1.27)) (justify left bottom))
   )
-  (label "VM" (at 33.02 96.52 0) (fields_autoplaced)
-    (effects (font (size 1.27 1.27)) (justify left bottom))
+  (label "VM" (at 20.32 114.3 180) (fields_autoplaced)
+    (effects (font (size 1.27 1.27)) (justify right bottom))
   )
   (label "SWDIO" (at 215.9 67.31 180) (fields_autoplaced)
@@
     (effects (font (size 1.27 1.27)) (justify left bottom))
   )
-  (label "IP" (at 33.02 88.9 0) (fields_autoplaced)
+  (label "IP" (at 45.72 114.3 0) (fields_autoplaced)
     (effects (font (size 1.27 1.27)) (justify left bottom))
   )
@@
     (effects (font (size 1.27 1.27)) (justify left bottom))
   )
-  (label "UN" (at 33.02 86.36 0) (fields_autoplaced)
+  (label "UN" (at 45.72 111.76 0) (fields_autoplaced)
     (effects (font (size 1.27 1.27)) (justify left bottom))
   )
@@
     (effects (font (size 1.27 1.27)) (justify left bottom))
   )
-  (label "Heater+" (at 33.02 99.06 0) (fields_autoplaced)
-    (effects (font (size 1.27 1.27)) (justify left bottom))
+  (label "Heater+" (at 20.32 116.84 180) (fields_autoplaced)
+    (effects (font (size 1.27 1.27)) (justify right bottom))
   )
   (label "SPI_SCK" (at 114.3 73.66 0) (fields_autoplaced)
@@
     (effects (font (size 1.27 1.27)) (justify left bottom))
   )
-  (label "Heater-" (at 33.02 93.98 0) (fields_autoplaced)
-    (effects (font (size 1.27 1.27)) (justify left bottom))
+  (label "Heater-" (at 20.32 111.76 180) (fields_autoplaced)
+    (effects (font (size 1.27 1.27)) (justify right bottom))
   )
   (label "SPI_NSS" (at 114.3 71.12 0) (fields_autoplaced)
@@
       (effects (font (size 1.27 1.27)))
     )
-    (property "Footprint" "Connector_PinHeader_1.00mm:PinHeader_2x10_P1.00mm_Vertical" (at 220.98 69.85 0)
+    (property "Footprint" "Connector_IDC:IDC-Header_2x10_P2.54mm_Vertical" (at 220.98 69.85 0)
       (effects (font (size 1.27 1.27)) hide)
     )
@@
     )
   )
+  (symbol (lib_id "MolexReceptacle 2x3:1053101106") (at 33.02 114.3 0) (unit 1)
+    (in_bom yes) (on_board yes) (dnp no) (fields_autoplaced)
+    (property "Reference" "J1" (at 33.02 104.14 0)
+      (effects (font (size 1.27 1.27)))
+    )
+    (property "Value" "2x3 O2 Connector" (at 33.02 106.68 0)
+      (effects (font (size 1.27 1.27)))
+    )
+    (property "Footprint" "CJ125 Circuit Data:MOLEX_1053101106" (at 33.02 114.3 0)
+      (effects (font (size 1.27 1.27)) (justify bottom) hide)
+    )
+    (property "Datasheet" "" (at 33.02 114.3 0)
+      (effects (font (size 1.27 1.27)) hide)
+    )
+    (property "MF" "Molex" (at 33.02 114.3 0)
+      (effects (font (size 1.27 1.27)) (justify bottom) hide)
+    )
+    (property "MAXIMUM_PACKAGE_HEIGHT" "10.51 mm" (at 33.02 114.3 0)
+      (effects (font (size 1.27 1.27)) (justify bottom) hide)
+    )
+    (property "Package" "None" (at 33.02 114.3 0)
+      (effects (font (size 1.27 1.27)) (justify bottom) hide)
+    )
+    (property "Price" "None" (at 33.02 114.3 0)
+      (effects (font (size 1.27 1.27)) (justify bottom) hide)
+    )
+    (property "Check_prices" "https://www.snapeda.com/parts/105310-1106/Molex/view-part/?ref=eda" (at 33.02 114.3 0)
+      (effects (font (size 1.27 1.27)) (justify bottom) hide)
+    )
+    (property "STANDARD" "Manufacturer Recommendations" (at 33.02 114.3 0)
+      (effects (font (size 1.27 1.27)) (justify bottom) hide)
+    )
+    (property "PARTREV" "H" (at 33.02 114.3 0)
+      (effects (font (size 1.27 1.27)) (justify bottom) hide)
+    )
+    (property "SnapEDA_Link" "https://www.snapeda.com/parts/105310-1106/Molex/view-part/?ref=snap" (at 33.02 114.3 0)
+      (effects (font (size 1.27 1.27)) (justify bottom) hide)
+    )
+    (property "MP" "105310-1106" (at 33.02 114.3 0)
+      (effects (font (size 1.27 1.27)) (justify bottom) hide)
+    )
+    (property "Purchase-URL" "https://www.snapeda.com/api/url_track_click_mouser/?unipart_id=1381131&manufacturer=Molex&part_name=105310-1106&search_term=1053101106" (at 33.02 114.3 0)
+      (effects (font (size 1.27 1.27)) (justify bottom) hide)
+    )
+    (property "Description" "\nConn Power HDR 6 POS 2.5mm Solder ST Thru-Hole 6 Terminal 1 Port Nano-Fit™ Tray\n" (at 33.02 114.3 0)
+      (effects (font (size 1.27 1.27)) (justify bottom) hide)
+    )
+    (property "Availability" "In Stock" (at 33.02 114.3 0)
+      (effects (font (size 1.27 1.27)) (justify bottom) hide)
+    )
+    (property "MANUFACTURER" "Molex" (at 33.02 114.3 0)
+      (effects (font (size 1.27 1.27)) (justify bottom) hide)
+    )
+    (pin "1")
+    (pin "2")
+    (pin "3")
+    (pin "4")
+    (pin "5")
+    (pin "6")
+    (instances
+      (project "CJ125 Circuit Design"
+        (path "/74f55849-6c80-40d8-a149-d776335dd88e"
+          (reference "J1") (unit 1)
+        )
+      )
+    )
+  )
   (symbol (lib_id "Device:C") (at 255.27 140.97 0) (unit 1)
     (in_bom yes) (on_board yes) (dnp no) (fields_autoplaced)
@@
         )
       )
-    )
-  )
-  (symbol (lib_id "Connector:Conn_01x06_Pin") (at 27.94 91.44 0) (unit 1)
-    (in_bom yes) (on_board yes) (dnp no) (fields_autoplaced)
-    (property "Reference" "J4" (at 28.575 81.28 0)
-      (effects (font (size 1.27 1.27)))
-    )
-    (property "Value" "1x6 O2 Connector" (at 28.575 83.82 0)
-      (effects (font (size 1.27 1.27)))
-    )
-    (property "Footprint" "Connector_PinHeader_1.00mm:PinHeader_1x06_P1.00mm_Vertical" (at 27.94 91.44 0)
-      (effects (font (size 1.27 1.27)) hide)
-    )
-    (property "Datasheet" "~" (at 27.94 91.44 0)
-      (effects (font (size 1.27 1.27)) hide)
-    )
-    (pin "1")
-    (pin "2")
-    (pin "3")
-    (pin "4")
-    (pin "5")
-    (pin "6")
-    (instances
-      (project "CJ125 Circuit Design"
-        (path "/74f55849-6c80-40d8-a149-d776335dd88e"
-          (reference "J4") (unit 1)
-        )
-      )
